Commit message: Created new core URFD

File: description/robot.urdf.xacro (robot description, xacro)
@@ -2,3 +2,4 @@
 <robot xmlns:xacro="http://www.ros.org/wiki/xacro"  name="robot">
     <xacro:include filename="robot_core.xacro" />
+    <xacro:include filename="gazebo_control.xacro" />
 </robot>

File: description/robot_core.xacro (robot description, xacro)
@@ -1,144 +1,96 @@
 <?xml version="1.0"?>
-    <robot xmlns:xacro="http://www.ros.org/wiki/xacro" >
-    <xacro:include filename="inertial_macros.xacro"/>
-    <!-- Define materials -->
-    <material name="grey">
-        <color rgba="0.5 0.5 0.5 1"/>
-    </material>
-    <material name="white">
-        <color rgba="1 1 1 1"/>
-    </material>
-    <material name="red">
-        <color rgba="1 0 0 1"/>
-    </material>
-    <material name="black">
-        <color rgba="0 0 0 1"/>
-    </material>
-    <!-- Define parameters -->
-    <xacro:property name="body_length" value="0.26"/>
-    <xacro:property name="body_width" value="0.22"/>
-    <xacro:property name="body_height" value="0.35"/>
-    <xacro:property name="wheel_radius" value="0.0325" />
-    <xacro:property name="wheel_length" value="0.035" />
-    <xacro:property name="material_density" value="1240" />
-    <xacro:property name="body_mass" value="0.6" />
-    <xacro:property name="wheel_mass" value="0.1" />
-    <!-- BASE LINK -->
-    <link name="base_link">
+<robot xmlns:xacro="http://ros.org/wiki/xacro" name="delivery_bot">
+  <!-- === Include inertial macros === -->
+  <xacro:include filename="inertial_macros.xacro"/>
+  <!-- === Parameters === -->
+  <xacro:property name="body_length" value="0.26"/>
+  <xacro:property name="body_width" value="0.22"/>
+  <xacro:property name="body_height" value="0.203"/>
+  <xacro:property name="wheel_to_body_bottom" value="0.01487"/>
+  <xacro:property name="body_center_z" value="${wheel_to_body_bottom + body_height / 2}"/>
+  <xacro:property name="wheel_radius" value="0.03675"/>
+  <xacro:property name="wheel_length" value="0.04"/>
+  <xacro:property name="wheel_mass" value="0.2"/>
+  <xacro:property name="wheel_rpy" value="${-pi/2} 0 0"/>
+  <xacro:property name="front_x" value="0.07268"/>
+  <xacro:property name="rear_x" value="-0.07268"/>
+  <xacro:property name="left_y" value="0.12606"/>
+  <xacro:property name="right_y" value="-0.12606"/>
+  <!-- === Base link at wheel axle height === -->
+  <link name="base_link"/>
+  <!-- === Body link === -->
+  <link name="body">
+    <visual>
+      <origin xyz="0 0 ${body_center_z}" rpy="0 0 0"/>
+      <geometry>
+        <box size="${body_length} ${body_width} ${body_height}"/>
+      </geometry>
+    </visual>
+    <collision>
+      <origin xyz="0 0 ${body_center_z}" rpy="0 0 0"/>
+      <geometry>
+        <box size="${body_length} ${body_width} ${body_height}"/>
+      </geometry>
+    </collision>
+    <xacro:inertial_box mass="1.0" x="${body_length}" y="${body_width}" z="${body_height}">
+      <origin xyz="0 0 ${body_center_z}" rpy="0 0 0"/>
+    </xacro:inertial_box>
+  </link>
+  <joint name="base_to_body" type="fixed">
+    <parent link="base_link"/>
+    <child link="body"/>
+    <origin xyz="0 0 0" rpy="0 0 0"/>
+  </joint>
+  <!-- === Wheel macro === -->
+  <xacro:macro name="wheel" params="name x y">
+    <link name="${name}">
+      <visual>
+        <origin xyz="0 0 0" rpy="${wheel_rpy}"/>
+        <geometry>
+          <cylinder radius="${wheel_radius}" length="${wheel_length}"/>
+        </geometry>
+      </visual>
+      <collision>
+        <origin xyz="0 0 0" rpy="${wheel_rpy}"/>
+        <geometry>
+          <cylinder radius="${wheel_radius}" length="${wheel_length}"/>
+        </geometry>
+      </collision>
+      <xacro:inertial_cylinder mass="${wheel_mass}" length="${wheel_length}" radius="${wheel_radius}">
+        <origin xyz="0 0 0" rpy="${wheel_rpy}"/>
+      </xacro:inertial_cylinder>
     </link>
-    <!--BODY LINK -->
-    <joint name="body_joint" type="fixed">
-        <parent link="base_link"/>
-        <child link="body"/>
-        <origin xyz="0 0 0"/>
+    <joint name="${name}_joint" type="continuous">
+      <parent link="base_link"/>
+      <child link="${name}"/>
+      <origin xyz="${x} ${y} 0" rpy="0 0 0"/>
+      <axis xyz="1 0 0"/>
     </joint>
-    <link name="body">
-        <visual>
-            <origin xyz="0 0 0"/>
-            <geometry>
-                <box size="${body_length} ${body_width} ${body_height}"/>
-            </geometry>
-            <material name="white"/>
-        </visual>
-        <collision>
-            <geometry>
-                <box size="${body_length} ${body_width} ${body_height}"/>
-            </geometry>
-        </collision>
-        <xacro:inertial_box mass="${body_mass}" x="0.53" y="0.42" z="0.42">
-            <origin xyz="0 0 0" rpy="0 0 0"/>
-        </xacro:inertial_box>
-    </link>
-    <!-- LEFT FRONT WHEEL LINK-->
-    <joint name="left_front_wheel_joint" type="continuous">
-        <parent link="base_link"/>
-        <child link="left_front_wheel"/>
-        <origin xyz="${body_length/2-1.2*wheel_radius} ${-body_width/2-wheel_length/2} ${-body_height/2}" rpy="${-pi/2} 0 0"/>
-        <axis xyz="0 0 1"/>
-    </joint>
-    <link name="left_front_wheel">
-        <visual>
-        <geometry>
-            <cylinder radius="${wheel_radius}" length="${wheel_length}"/>
-        </geometry>
-        <material name="black"/>
-        </visual>
-        <collision>
-            <geometry>
-                <cylinder radius="${wheel_radius}" length="${wheel_length}"/>
-            </geometry>
-        </collision>
-        <xacro:inertial_cylinder mass="${wheel_mass}" length="${wheel_length}" radius="${wheel_radius}">
-            <origin xyz="0 0 0" rpy="0 0 0"/>
-        </xacro:inertial_cylinder>
-    </link>
-    <!-- RIGHT FRONT WHEEL LINK-->
-    <joint name="right_front_wheel_joint" type="continuous">
-        <parent link="base_link"/>
-        <child link="right_front_wheel"/>
-        <origin xyz="${body_length/2-1.2*wheel_radius} ${body_width/2+wheel_length/2} ${-body_height/2}" rpy="${pi/2} 0 0"/>
-        <axis xyz="0 0 -1"/>
-    </joint>
-    <link name="right_front_wheel">
-        <visual>
-        <geometry>
-            <cylinder radius="${wheel_radius}" length="${wheel_length}"/>
-        </geometry>
-        <material name="black"/>
-        </visual>
-        <collision>
-            <geometry>
-                <cylinder radius="${wheel_radius}" length="${wheel_length}"/>
-            </geometry>
-        </collision>
-        <xacro:inertial_cylinder mass="${wheel_mass}" length="${wheel_length}" radius="${wheel_radius}">
-            <origin xyz="0 0 0" rpy="0 0 0"/>
-        </xacro:inertial_cylinder>
-    </link>
-    <!-- LEFT REAR WHEEL LINK-->
-    <joint name="left_rear_wheel_joint" type="continuous">
-        <parent link="base_link"/>
-        <child link="left_rear_wheel"/>
-        <origin xyz="${-body_length/2+1.2*wheel_radius} ${-body_width/2-wheel_length/2} ${-body_height/2}" rpy="${-pi/2} 0 0"/>
-        <axis xyz="0 0 1"/>
-    </joint>
-    <link name="left_rear_wheel">
-        <visual>
-        <geometry>
-            <cylinder radius="${wheel_radius}" length="${wheel_length}"/>
-        </geometry>
-        <material name="black"/>
-        </visual>
-        <collision>
-            <geometry>
-                <cylinder radius="${wheel_radius}" length="${wheel_length}"/>
-            </geometry>
-        </collision>
-        <xacro:inertial_cylinder mass="${wheel_mass}" length="${wheel_length}" radius="${wheel_radius}">
-            <origin xyz="0 0 0" rpy="0 0 0"/>
-        </xacro:inertial_cylinder>
-    </link>
-      <!-- RIGHT REAR WHEEL LINK-->
-    <joint name="right_rear_wheel_joint" type="continuous">
-        <parent link="base_link"/>
-        <child link="right_rear_wheel"/>
-        <origin xyz="${-body_length/2+1.2*wheel_radius} ${body_width/2+wheel_length/2} ${-body_height/2}" rpy="${-pi/2} 0 0"/>
-        <axis xyz="0 0 1"/>
-    </joint>
-    <link name="right_rear_wheel">
-        <visual>
-        <geometry>
-            <cylinder radius="${wheel_radius}" length="${wheel_length}"/>
-        </geometry>
-        <material name="black"/>
-        </visual>
-        <collision>
-            <geometry>
-                <cylinder radius="${wheel_radius}" length="${wheel_length}"/>
-            </geometry>
-        </collision>
-        <xacro:inertial_cylinder mass="${wheel_mass}" length="${wheel_length}" radius="${wheel_radius}">
-            <origin xyz="0 0 0" rpy="0 0 0"/>
-        </xacro:inertial_cylinder>
-    </link>
+  </xacro:macro>
+  <!-- === Wheels === -->
+  <xacro:wheel name="front_left_wheel"  x="${front_x}" y="${left_y}"/>
+  <xacro:wheel name="front_right_wheel" x="${front_x}" y="${right_y}"/>
+  <xacro:wheel name="rear_left_wheel"   x="${rear_x}"  y="${left_y}"/>
+  <xacro:wheel name="rear_right_wheel"  x="${rear_x}"  y="${right_y}"/>
+  <!-- === Gazebo tags for wheel appearance and multipliers === -->
+  <gazebo reference="front_left_wheel">
+    <material>Gazebo/Black</material>
+    <mul1>0.1</mul1>
+    <mul2>0.1</mul2>
+  </gazebo>
+  <gazebo reference="front_right_wheel">
+    <material>Gazebo/Black</material>
+    <mul1>0.1</mul1>
+    <mul2>0.1</mul2>
+  </gazebo>
+  <gazebo reference="rear_left_wheel">
+    <material>Gazebo/Black</material>
+    <mul1>0.1</mul1>
+    <mul2>0.1</mul2>
+  </gazebo>
+  <gazebo reference="rear_right_wheel">
+    <material>Gazebo/Black</material>
+    <mul1>0.1</mul1>
+    <mul2>0.1</mul2>
+  </gazebo>
 </robot>
