Commit message: added gazebo control and obstacles world

File: description/gazebo_control.xacro (robot description, xacro)
@@ -2,17 +2,17 @@
 <robot xmlns:xacro="http://www.ros.org/wiki/xacro">
     <gazebo>
-        <plugin name="differential_drive" filename="libgazebo_ros_diff_drive.so">
-            <!-- <ros>
+        <plugin name="diff_drive_controller" filename="libgazebo_ros_diff_drive.so">
+            <ros>
                 <namespace> </namespace>
-            </ros> -->
+            </ros>
             <!-- Wheel Information -->
             <num_wheel_pairs>2</num_wheel_pairs>
-            <left_joint>front_left_wheel_joint</left_joint>
-            <left_joint>rear_left_wheel_joint</left_joint>
-            <right_joint>front_right_wheel_joint</right_joint>
-            <right_joint>rear_right_wheel_joint</right_joint>
+            <left_joint>left_front_wheel_joint</left_joint>
+            <left_joint>left_rear_wheel_joint</left_joint>
+            <right_joint>right_front_wheel_joint</right_joint>
+            <right_joint>right_rear_wheel_joint</right_joint>
             <!--Kinematics-->
-            <wheel_separation>0.25212</wheel_separation>
-            <wheel_diameter>0.0735</wheel_diameter>
+            <wheel_separation>0.1228</wheel_separation>
+            <wheel_diameter>${2*wheel_radius}</wheel_diameter>
             <!-- Limits -->
             <max_wheel_torque>1000</max_wheel_torque>
@@ -25,8 +25,8 @@
             <odometry_frame>odom</odometry_frame>
             <robot_base_frame>base_link</robot_base_frame>
-            <!-- <publish_wheel_joint_state>true</publish_wheel_joint_state>
+            <publish_wheel_joint_state>true</publish_wheel_joint_state>
             <covariance_x>0.001</covariance_x>
             <covariance_y>0.001</covariance_y>
-            <covariance_yaw>0.01</covariance_yaw> -->
+            <covariance_yaw>0.01</covariance_yaw>
         </plugin>
     </gazebo>

File: description/inertial_macros.xacro (robot description, xacro)
@@ -3,8 +3,8 @@
     <!-- Specify some standard inertial calculations https://en.wikipedia.org/wiki/List_of_moments_of_inertia -->
     <!-- These make use of xacro's mathematical functionality -->
-    <xacro:macro name="inertial_box" params="mass x y z *origin">
+   <xacro:macro name="inertial_box" params="mass x y z *origin">
         <inertial>
             <xacro:insert_block name="origin"/>
-            <mass value="${mass}" />
+            <mass value="${body_mass}" />
             <inertia ixx="${(1/12) * mass * (y*y+z*z)}" ixy="0.0" ixz="0.0"
                     iyy="${(1/12) * mass * (x*x+z*z)}" iyz="0.0"
@@ -15,5 +15,5 @@
         <inertial>
             <xacro:insert_block name="origin"/>
-            <mass value="${mass}" />
+            <mass value="${wheel_mass}" />
             <inertia ixx="${(1/12) * mass * (3*radius*radius + length*length)}" ixy="0.0" ixz="0.0"
                     iyy="${(1/12) * mass * (3*radius*radius + length*length)}" iyz="0.0"

File: description/robot.urdf.xacro (robot description, xacro)
@@ -2,4 +2,8 @@
 <robot xmlns:xacro="http://www.ros.org/wiki/xacro"  name="robot">
     <xacro:include filename="robot_core.xacro" />
+    <!-- <xacro:include filename="ros2_control.xacro" /> -->
     <xacro:include filename="gazebo_control.xacro" />
+    <!-- <xacro:include filename="lidar.xacro" /> -->
+    <!-- <xacro:include filename="camera.xacro" /> -->
+    <!-- <xacro:include filename="depth_camera.xacro" /> -->
 </robot>

File: description/robot_core.xacro (robot description, xacro)
@@ -1,7 +1,20 @@
 <?xml version="1.0"?>
 <robot xmlns:xacro="http://ros.org/wiki/xacro" name="delivery_bot">
-  <!-- === Include inertial macros === -->
+  <!-- Include macros -->
   <xacro:include filename="inertial_macros.xacro"/>
-  <!-- === Parameters === -->
+  <!-- Materials -->
+  <material name="grey">
+    <color rgba="0.5 0.5 0.5 1"/>
+  </material>
+  <material name="white">
+    <color rgba="1 1 1 1"/>
+  </material>
+  <material name="red">
+    <color rgba="1 0 0 1"/>
+  </material>
+  <material name="black">
+    <color rgba="0 0 0 1"/>
+  </material>
+  <!-- Parameters -->
   <xacro:property name="body_length" value="0.26"/>
   <xacro:property name="body_width" value="0.22"/>
@@ -9,88 +22,152 @@
   <xacro:property name="wheel_to_body_bottom" value="0.01487"/>
   <xacro:property name="body_center_z" value="${wheel_to_body_bottom + body_height / 2}"/>
-  <xacro:property name="wheel_radius" value="0.03675"/>
-  <xacro:property name="wheel_length" value="0.04"/>
-  <xacro:property name="wheel_mass" value="0.2"/>
-  <xacro:property name="wheel_rpy" value="${-pi/2} 0 0"/>
-  <xacro:property name="front_x" value="0.07268"/>
-  <xacro:property name="rear_x" value="-0.07268"/>
-  <xacro:property name="left_y" value="0.12606"/>
-  <xacro:property name="right_y" value="-0.12606"/>
-  <!-- === Base link at wheel axle height === -->
-  <link name="base_link"/>
-  <!-- === Body link === -->
-  <link name="body">
+  <xacro:property name="wheel_radius" value="0.034"/>
+  <xacro:property name="wheel_width" value="0.0256"/>
+  <xacro:property name="body_mass" value="0.8"/>
+  <xacro:property name="wheel_mass" value="0.1"/>
+  <xacro:property name="material_density" value="1180" />
+  <!-- Base link -->
+  <link name="base_link" />
+  <!-- Chassis joint -->
+  <joint name="chassis_joint" type="fixed">
+    <parent link="base_link"/>
+    <child link="chassis"/>
+    <origin xyz="0 0 0"/>
+  </joint>
+  <!-- Chassis link -->
+  <link name="chassis">
     <visual>
-      <origin xyz="0 0 ${body_center_z}" rpy="0 0 0"/>
+      <origin xyz="0 0 0" />
       <geometry>
-        <box size="${body_length} ${body_width} ${body_height}"/>
+        <box size="${body_length} ${body_width} ${body_height}" />
       </geometry>
+      <material name="white" />
     </visual>
     <collision>
-      <origin xyz="0 0 ${body_center_z}" rpy="0 0 0"/>
+      <origin xyz="0 0 0" />
       <geometry>
-        <box size="${body_length} ${body_width} ${body_height}"/>
+        <box size="${body_length} ${body_width} ${body_height}" />
       </geometry>
     </collision>
-    <xacro:inertial_box mass="1.0" x="${body_length}" y="${body_width}" z="${body_height}">
-      <origin xyz="0 0 ${body_center_z}" rpy="0 0 0"/>
+    <xacro:inertial_box mass="${body_mass}" x="${body_length}" y="${body_width}" z="${body_height}">
+      <origin xyz="0 0 0" />
     </xacro:inertial_box>
   </link>
-  <joint name="base_to_body" type="fixed">
+  <gazebo reference="chassis">
+    <material>Gazebo/White</material>
+    <mu1>0.1</mu1>
+    <mu2>0.1</mu2>
+  </gazebo>
+  <!-- LEFT FRONT WHEEL LINK -->
+  <joint name="left_front_wheel_joint" type="continuous">
     <parent link="base_link"/>
-    <child link="body"/>
-    <origin xyz="0 0 0" rpy="0 0 0"/>
+    <child link="left_front_wheel"/>
+    <origin xyz="${body_length/2-1.2*wheel_radius} ${-body_width/2-wheel_width/2} ${-body_height/2}" rpy="-${pi/2} 0 0"/>
+    <axis xyz="0 0 1"/>
   </joint>
-  <!-- === Wheel macro === -->
-  <xacro:macro name="wheel" params="name x y">
-    <link name="${name}">
-      <visual>
-        <origin xyz="0 0 0" rpy="${wheel_rpy}"/>
-        <geometry>
-          <cylinder radius="${wheel_radius}" length="${wheel_length}"/>
-        </geometry>
-      </visual>
-      <collision>
-        <origin xyz="0 0 0" rpy="${wheel_rpy}"/>
-        <geometry>
-          <cylinder radius="${wheel_radius}" length="${wheel_length}"/>
-        </geometry>
-      </collision>
-      <xacro:inertial_cylinder mass="${wheel_mass}" length="${wheel_length}" radius="${wheel_radius}">
-        <origin xyz="0 0 0" rpy="${wheel_rpy}"/>
-      </xacro:inertial_cylinder>
-    </link>
-    <joint name="${name}_joint" type="continuous">
-      <parent link="base_link"/>
-      <child link="${name}"/>
-      <origin xyz="${x} ${y} 0" rpy="0 0 0"/>
-      <axis xyz="1 0 0"/>
-    </joint>
-  </xacro:macro>
-  <!-- === Wheels === -->
-  <xacro:wheel name="front_left_wheel"  x="${front_x}" y="${left_y}"/>
-  <xacro:wheel name="front_right_wheel" x="${front_x}" y="${right_y}"/>
-  <xacro:wheel name="rear_left_wheel"   x="${rear_x}"  y="${left_y}"/>
-  <xacro:wheel name="rear_right_wheel"  x="${rear_x}"  y="${right_y}"/>
-  <!-- === Gazebo tags for wheel appearance and multipliers === -->
-  <gazebo reference="front_left_wheel">
+  <link name="left_front_wheel">
+    <visual>
+      <geometry>
+        <cylinder radius="${wheel_radius}" length="${wheel_width}"/>
+      </geometry>
+      <material name="black"/>
+    </visual>
+    <collision>
+      <geometry>
+        <cylinder radius="${wheel_radius}" length="${wheel_width}"/>
+      </geometry>
+    </collision>
+    <xacro:inertial_cylinder mass="${wheel_mass}" length="${wheel_width}" radius="${wheel_radius}">
+      <origin xyz="0 0 0" rpy="0 0 0" />
+    </xacro:inertial_cylinder>
+  </link>
+  <gazebo reference="left_front_wheel">
     <material>Gazebo/Black</material>
-    <mul1>0.1</mul1>
-    <mul2>0.1</mul2>
+    <mu1>0.1</mu1>
+    <mu2>0.1</mu2>
   </gazebo>
-  <gazebo reference="front_right_wheel">
+  <!-- RIGHT FRONT WHEEL LINK -->
+  <joint name="right_front_wheel_joint" type="continuous">
+    <parent link="base_link"/>
+    <child link="right_front_wheel"/>
+    <origin xyz="${body_length/2-1.2*wheel_radius} ${body_width/2+wheel_width/2} ${-body_height/2}" rpy="${pi/2} 0 0"/>
+    <axis xyz="0 0 -1"/>
+  </joint>
+  <link name="right_front_wheel">
+    <visual>
+      <geometry>
+        <cylinder radius="${wheel_radius}" length="${wheel_width}"/>
+      </geometry>
+      <material name="black"/>
+    </visual>
+    <collision>
+      <geometry>
+        <cylinder radius="${wheel_radius}" length="${wheel_width}"/>
+      </geometry>
+    </collision>
+     <xacro:inertial_cylinder mass="${wheel_mass}" length="${wheel_width}" radius="${wheel_radius}">
+      <origin xyz="0 0 0" rpy="0 0 0" />
+    </xacro:inertial_cylinder>
+  </link>
+  <gazebo reference="right_front_wheel">
     <material>Gazebo/Black</material>
-    <mul1>0.1</mul1>
-    <mul2>0.1</mul2>
+    <mu1>0.1</mu1>
+    <mu2>0.1</mu2>
   </gazebo>
-  <gazebo reference="rear_left_wheel">
+ <!-- LEFT REAR WHEEL LINK -->
+  <joint name="left_rear_wheel_joint" type="continuous">
+    <parent link="base_link"/>
+    <child link="left_rear_wheel"/>
+    <origin xyz="${-body_length/2+1.2*wheel_radius} ${-body_width/2-wheel_width/2} ${-body_height/2}" rpy="-${pi/2} 0 0"/>
+    <axis xyz="0 0 1"/>
+  </joint>
+  <link name="left_rear_wheel">
+    <visual>
+      <geometry>
+        <cylinder radius="${wheel_radius}" length="${wheel_width}"/>
+      </geometry>
+      <material name="black"/>
+    </visual>
+    <collision>
+      <geometry>
+        <cylinder radius="${wheel_radius}" length="${wheel_width}"/>
+      </geometry>
+    </collision>
+     <xacro:inertial_cylinder mass="${wheel_mass}" length="${wheel_width}" radius="${wheel_radius}">
+      <origin xyz="0 0 0" rpy="0 0 0" />
+    </xacro:inertial_cylinder>
+  </link>
+  <gazebo reference="left_rear_wheel">
     <material>Gazebo/Black</material>
-    <mul1>0.1</mul1>
-    <mul2>0.1</mul2>
+    <mu1>0.1</mu1>
+    <mu2>0.1</mu2>
   </gazebo>
-  <gazebo reference="rear_right_wheel">
+  <!-- RIGHT REAR WHEEL LINK -->
+  <joint name="right_rear_wheel_joint" type="continuous">
+    <parent link="base_link"/>
+    <child link="right_rear_wheel"/>
+    <origin xyz="${-body_length/2+1.2*wheel_radius} ${body_width/2+wheel_width/2} ${-body_height/2}" rpy="${pi/2} 0 0"/>
+    <axis xyz="0 0 -1"/>
+  </joint>
+  <link name="right_rear_wheel">
+    <visual>
+      <geometry>
+        <cylinder radius="${wheel_radius}" length="${wheel_width}"/>
+      </geometry>
+      <material name="black"/>
+    </visual>
+    <collision>
+      <geometry>
+        <cylinder radius="${wheel_radius}" length="${wheel_width}"/>
+      </geometry>
+    </collision>
+     <xacro:inertial_cylinder mass="${wheel_mass}" length="${wheel_width}" radius="${wheel_radius}">
+      <origin xyz="0 0 0" rpy="0 0 0" />
+    </xacro:inertial_cylinder>
+  </link>
+  <gazebo reference="right_rear_wheel">
     <material>Gazebo/Black</material>
-    <mul1>0.1</mul1>
-    <mul2>0.1</mul2>
+    <mu1>0.1</mu1>
+    <mu2>0.1</mu2>
   </gazebo>
 </robot>
